File: kapuki-cursen-hw.sch (KiCad schematic (older format))
At the start: 30 parts, among them J1 Conn_01x02, J2 Conn_01x02, J3 Conn_01x01, J4 Conn_01x01, J5 Conn_01x01, J6 Conn_01x01, J7 Conn_01x06, J8 Conn_01x05, U1 MIC5235, U2 MAX4081S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

Commit message: Routing rev.1
Parts:
- R2: footprint Resistor_SMD:R_0201_0603Metric -> Resistor_SMD:R_0402_1005Metric
- R3: renamed from R6; footprint Resistor_SMD:R_0201_0603Metric -> Resistor_SMD:R_0402_1005Metric
- R4: renamed from R3; footprint Resistor_SMD:R_0201_0603Metric -> Resistor_SMD:R_0402_1005Metric
- R5: renamed from R4; footprint Resistor_SMD:R_0201_0603Metric -> Resistor_SMD:R_0402_1005Metric
- R6: renamed from R5; footprint Resistor_SMD:R_0201_0603Metric -> Resistor_SMD:R_0402_1005Metric
Connections:
- net labels added: LED, VCCA
- wire segments 124 -> 125
- no-connect marks 14 -> 13
Changed lines of the file:
@@
 F 0 "R2" V 3593 2400 50  0000 C CNN
 F 1 "R" V 3684 2400 50  0000 C CNN
-F 2 "Resistor_SMD:R_0201_0603Metric" V 3730 2400 50  0001 C CNN
+F 2 "Resistor_SMD:R_0402_1005Metric" V 3730 2400 50  0001 C CNN
 F 3 "~" H 3800 2400 50  0001 C CNN
 	1    3800 2400
@@
 	1550 5850 1400 5850
 $Comp
-L kapuki:STM32G431KBUx U3
-U 1 1 5DD32172
-P 8200 3150
-F 0 "U3" H 7850 4000 50  0000 C CNN
-F 1 "STM32G431KBUx" H 8650 2200 50  0000 C CNN
-F 2 "Package_DFN_QFN:QFN-32-1EP_5x5mm_P0.5mm_EP3.45x3.45mm" H 7800 2250 50  0001 R CNN
-F 3 "https://www.st.com/resource/en/datasheet/stm32g431c6.pdf" H 8200 3150 50  0001 C CNN
-	1    8200 3150
-	1    0    0    -1
-$EndComp
-$Comp
-L power:GND #PWR010
+L power:GND #PWR012
 U 1 1 5DD36699
 P 8300 4250
-F 0 "#PWR010" H 8300 4000 50  0001 C CNN
+F 0 "#PWR012" H 8300 4000 50  0001 C CNN
 F 1 "GND" H 8305 4077 50  0000 C CNN
 F 2 "" H 8300 4250 50  0001 C CNN
@@
 Wire Wire Line
 	8500 1650 8500 1700
-Wire Wire Line
-	8500 1650 8300 1650
 Connection ~ 8500 1650
 Wire Wire Line
@@
 	8100 2200 8100 1650
 $Comp
-L power:GND #PWR011
+L power:GND #PWR013
 U 1 1 5DD47314
 P 8900 2100
-F 0 "#PWR011" H 8900 1850 50  0001 C CNN
+F 0 "#PWR013" H 8900 1850 50  0001 C CNN
 F 1 "GND" H 8905 1927 50  0000 C CNN
 F 2 "" H 8900 2100 50  0001 C CNN
@@
 $EndComp
 $Comp
-L power:GND #PWR08
+L power:GND #PWR09
 U 1 1 5DD47B4D
 P 7250 2100
-F 0 "#PWR08" H 7250 1850 50  0001 C CNN
+F 0 "#PWR09" H 7250 1850 50  0001 C CNN
 F 1 "GND" H 7255 1927 50  0000 C CNN
 F 2 "" H 7250 2100 50  0001 C CNN
@@
 Text Label 8750 3350 0    50   ~ 0
 RXTX
+Text Label 8750 3750 0    50   ~ 0
+SWCLK
 Text Label 8750 3850 0    50   ~ 0
-SWCLK
-Text Label 8750 3950 0    50   ~ 0
 SWDIO
-Wire Wire Line
-	8700 3950 9250 3950
 Wire Wire Line
 	8700 3850 9250 3850
@@
 MOTORPULSE
 $Comp
-L Device:R R5
+L Device:R R6
 U 1 1 5DD70BDC
 P 10200 3150
-F 0 "R5" H 10130 3104 50  0000 R CNN
+F 0 "R6" H 10130 3104 50  0000 R CNN
 F 1 "R" H 10130 3195 50  0000 R CNN
-F 2 "Resistor_SMD:R_0201_0603Metric" V 10130 3150 50  0001 C CNN
+F 2 "Resistor_SMD:R_0402_1005Metric" V 10130 3150 50  0001 C CNN
 F 3 "~" H 10200 3150 50  0001 C CNN
 	1    10200 3150
@@
 Wire Wire Line
 	3950 6400 4250 6400
-NoConn ~ 8700 3750
 NoConn ~ 8700 3650
-NoConn ~ 8700 3550
 NoConn ~ 8700 3450
 NoConn ~ 7700 2600
@@
 	7750 5650 8150 5650
 $Comp
-L power:GND #PWR09
+L power:GND #PWR011
 U 1 1 5DD35CC2
 P 8050 5450
-F 0 "#PWR09" H 8050 5200 50  0001 C CNN
+F 0 "#PWR011" H 8050 5200 50  0001 C CNN
 F 1 "GND" V 8050 5250 50  0000 C CNN
 F 2 "" H 8050 5450 50  0001 C CNN
@@
 Connection ~ 8500 1450
 $Comp
-L Device:R R3
+L Device:R R4
 U 1 1 5DD3EEEA
 P 9700 2450
-F 0 "R3" H 9630 2404 50  0000 R CNN
+F 0 "R4" H 9630 2404 50  0000 R CNN
 F 1 "R" H 9630 2495 50  0000 R CNN
-F 2 "Resistor_SMD:R_0201_0603Metric" V 9630 2450 50  0001 C CNN
+F 2 "Resistor_SMD:R_0402_1005Metric" V 9630 2450 50  0001 C CNN
 F 3 "~" H 9700 2450 50  0001 C CNN
 	1    9700 2450
@@
 $EndComp
 $Comp
-L Device:R R4
+L Device:R R5
 U 1 1 5DD3F6D0
 P 9700 2850
-F 0 "R4" H 9630 2804 50  0000 R CNN
+F 0 "R5" H 9630 2804 50  0000 R CNN
 F 1 "R" H 9630 2895 50  0000 R CNN
-F 2 "Resistor_SMD:R_0201_0603Metric" V 9630 2850 50  0001 C CNN
+F 2 "Resistor_SMD:R_0402_1005Metric" V 9630 2850 50  0001 C CNN
 F 3 "~" H 9700 2850 50  0001 C CNN
 	1    9700 2850
@@
 $EndComp
 $Comp
-L power:GND #PWR012
+L power:GND #PWR014
 U 1 1 5DD3FBEC
 P 9700 3075
-F 0 "#PWR012" H 9700 2825 50  0001 C CNN
+F 0 "#PWR014" H 9700 2825 50  0001 C CNN
 F 1 "GND" H 9705 2902 50  0000 C CNN
 F 2 "" H 9700 3075 50  0001 C CNN
@@
 	9700 2650 9700 2600
 NoConn ~ 8150 5650
-Wire Wire Line
-	8300 2250 8300 1650
 $Comp
 L Connector_Generic:Conn_01x02 J1
@@
 $EndComp
 $Comp
-L Device:R R6
+L Device:R R3
 U 1 1 5DDCAC4A
 P 6400 3200
-F 0 "R6" H 6330 3154 50  0000 R CNN
+F 0 "R3" H 6330 3154 50  0000 R CNN
 F 1 "R" H 6330 3245 50  0000 R CNN
-F 2 "Resistor_SMD:R_0201_0603Metric" V 6330 3200 50  0001 C CNN
+F 2 "Resistor_SMD:R_0402_1005Metric" V 6330 3200 50  0001 C CNN
 F 3 "~" H 6400 3200 50  0001 C CNN
 	1    6400 3200
@@
 $EndComp
 Wire Wire Line
-	7700 3450 6400 3450
-Wire Wire Line
-	6400 3450 6400 3350
-Wire Wire Line
 	6400 3050 6400 2975
 $Comp
-L power:VCC #PWR013
+L power:VCC #PWR08
 U 1 1 5DDD674D
 P 6400 2600
-F 0 "#PWR013" H 6400 2450 50  0001 C CNN
+F 0 "#PWR08" H 6400 2450 50  0001 C CNN
 F 1 "VCC" H 6417 2773 50  0000 C CNN
 F 2 "" H 6400 2600 50  0001 C CNN
@@
 $EndComp
 $Comp
-L power:VCC #PWR014
+L power:VCC #PWR010
 U 1 1 5DDD6BD3
 P 7650 1400
-F 0 "#PWR014" H 7650 1250 50  0001 C CNN
+F 0 "#PWR010" H 7650 1250 50  0001 C CNN
 F 1 "VCC" H 7667 1573 50  0000 C CNN
 F 2 "" H 7650 1400 50  0001 C CNN
@@
 Wire Wire Line
 	6400 2675 6400 2600
+Text Label 8600 1650 0    50   ~ 0
+VCCA
+Wire Wire Line
+	8300 2250 8300 1650
+Wire Wire Line
+	8300 1650 8500 1650
+$Comp
+L kapuki:STM32G431KBUx U3
+U 1 1 5DE1D368
+P 8200 3150
+F 0 "U3" H 8200 4231 50  0000 C CNN
+F 1 "STM32G431KBUx" H 8200 4140 50  0000 C CNN
+F 2 "Package_DFN_QFN:QFN-32-1EP_5x5mm_P0.5mm_EP3.45x3.45mm" H 7800 2250 50  0001 R CNN
+F 3 "https://www.st.com/resource/en/datasheet/stm32g431c6.pdf" H 8200 3150 50  0001 C CNN
+	1    8200 3150
+	1    0    0    -1
+$EndComp
+Wire Wire Line
+	8700 3750 9250 3750
+NoConn ~ 8700 3950
+Wire Wire Line
+	6400 3550 6825 3550
+Wire Wire Line
+	6400 3350 6400 3550
+Text Label 6625 3550 0    50   ~ 0
+LED
+Wire Wire Line
+	8700 3550 9250 3550
+Text Label 8750 3550 0    50   ~ 0
+LED
 $EndSCHEMATC

Commit message: Rev. 2
Parts:
- removed D2, D4: BZT52H-C3V3, Diode_SMD:D_SOD-123F, symbol Diode:BZT52Bxx
- removed J3, J4, J5: Conn_01x01, Connector_PinSocket_2.54mm:PinSocket_1x01_P2.54mm_Vertical, symbol Connector_Generic:Conn_01x01
- added C10: 2.2uF, Capacitor_SMD:C_0402_1005Metric, symbol Device:C
- added C11, C9: 100nF, Capacitor_SMD:C_0402_1005Metric, symbol Device:C
- added J3: Conn_01x03, Connector_PinHeader_2.54mm:PinHeader_1x03_P2.54mm_Vertical, symbol Connector_Generic:Conn_01x03
- added R7: 50, Resistor_SMD:R_0402_1005Metric, symbol Device:R
- added R8: 10k, Resistor_SMD:R_0402_1005Metric, symbol Device:R
- added U4: MCP1501, Package_TO_SOT_SMD:SOT-23-6, symbol kapuki:MCP1501
- C3: value C -> 100pF
- C8: value 100nF -> 10nF
- FB1: value Ferrite_Bead -> 120ohm GHz
- R1: value R_Shunt -> 0.0002 1% 12W
- R2: value R -> 1k
- R4: value R -> 38k3 0.1%
- R5: value R -> 2k4 0.1%
Connections:
- net labels added: +3V3, IMEAS, UMEAS, VDDA, ~RESET~
- net labels removed: CURRMEAS, EXT6, LED, NRESET, VCCA, VCCIN
- wire segments 125 -> 143
- no-connect marks 13 -> 11
Other:
- note added: "Absolute maximum ratings\n———————————————————\nMax. battery input voltage: 50V (12S)\nMax. current: 100A\n\nDC characteristics:\n———————————————————\nInput power supply: 4-10V\nPower consuption: 100mA"
- note added: "BLDC motor RPM sensor"
- note added: "Battery Current and Voltage measurement"
- note added: "Bourns CSS2H-3920R-L200FE"
- note added: "Extension port"
- note added: "Power supply & Jeti EX bus interface"
- note added: "SWD programming\n interface"
- note added: "Voltage reference and power supply for CPU Analog section"
- moved on the sheet: C1, C2, C3, C4, C5, C6, C7, C8, D1, D3, FB1, J1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

Commit message: Add precision voltage reference
Parts:
- R3: value R -> 1k
- R6: value R -> 4k7
Other:
- note added: "Absolute maximum ratings\n———————————————————\nMax. battery input voltage: 50V (12S)\nMax. current: 60A\n\nDC characteristics:\n———————————————————\nInput power supply: 4-10V\nPower consuption: 100mA"
- note removed: "Absolute maximum ratings\n———————————————————\nMax. battery input voltage: 50V (12S)\nMax. current: 100A\n\nDC characteristics:\n———————————————————\nInput power supply: 4-10V\nPower consuption: 100mA"
Changed lines of the file:
@@
 encoding utf-8
 Sheet 1 1
-Title "100A RC precision current sensor"
-Date "2020-01-29"
+Title "60A RC precision current sensor"
+Date "2020-01-31"
 Rev "2"
 Comp "bodrico.com"
@@
 P 10350 3050
 F 0 "R3" H 10280 3004 50  0000 R CNN
-F 1 "R" H 10280 3095 50  0000 R CNN
+F 1 "1k" H 10280 3095 50  0000 R CNN
 F 2 "Resistor_SMD:R_0402_1005Metric" V 10280 3050 50  0001 C CNN
 F 3 "~" H 10350 3050 50  0001 C CNN
@@
 P 9650 2900
 F 0 "R6" H 9580 2854 50  0000 R CNN
-F 1 "R" H 9580 2945 50  0000 R CNN
+F 1 "4k7" H 9580 2945 50  0000 R CNN
 F 2 "Resistor_SMD:R_0402_1005Metric" V 9580 2900 50  0001 C CNN
 F 3 "~" H 9650 2900 50  0001 C CNN
@@
 BLDC motor RPM sensor
 Text Notes 3650 1700 0    55   ~ 11
-Absolute maximum ratings\n———————————————————\nMax. battery input voltage: 50V (12S)\nMax. current: 100A\n\nDC characteristics:\n———————————————————\nInput power supply: 4-10V\nPower consuption: 100mA
+Absolute maximum ratings\n———————————————————\nMax. battery input voltage: 50V (12S)\nMax. current: 60A\n\nDC characteristics:\n———————————————————\nInput power supply: 4-10V\nPower consuption: 100mA
 Wire Notes Line style solid
 	3550 800  5400 800
@@
 	10100 5600 10050 5600
 $Comp
-L power:+3V3 #PWR?
+L power:+3V3 #PWR0110
 U 1 1 5E75D595
 P 8200 4950
-F 0 "#PWR?" H 8200 4800 50  0001 C CNN
+F 0 "#PWR0110" H 8200 4800 50  0001 C CNN
 F 1 "+3V3" H 8215 5123 50  0000 C CNN
 F 2 "" H 8200 4950 50  0001 C CNN

Commit message: Fix SWD connector and servo connector
Parts:
- C9: value 100nF -> 2.2uF
- R1: value 0.0002 1% 12W -> 0.0002ohm 1% 12W
- R7: value 50 -> 1k
Other:
- note added: "Absolute maximum ratings\n———————————————————\nMax. battery input voltage: 50V (12S)\nMax. current: 60A\n\nDC characteristics:\n———————————————————\nInput power supply: 4-10V\nPower consuption: 20mA"
- note removed: "Absolute maximum ratings\n———————————————————\nMax. battery input voltage: 50V (12S)\nMax. current: 60A\n\nDC characteristics:\n———————————————————\nInput power supply: 4-10V\nPower consuption: 100mA"
Changed lines of the file:
@@
 EESchema Schematic File Version 4
+LIBS:kapuki-cursen-hw-cache
 EELAYER 30 0
 EELAYER END
@@
 Sheet 1 1
 Title "60A RC precision current sensor"
-Date "2020-01-31"
-Rev "2"
+Date "2020-02-23"
+Rev "3"
 Comp "bodrico.com"
 Comment1 "bodri@bodrico.com"
@@
 P 2000 2600
 F 0 "R1" H 1912 2646 50  0000 R CNN
-F 1 "0.0002 1% 12W" H 1912 2555 50  0000 R CNN
+F 1 "0.0002ohm 1% 12W" H 1912 2555 50  0000 R CNN
 F 2 "local:Bourns_ CSS2H" V 1930 2600 50  0001 C CNN
 F 3 "~" H 2000 2600 50  0001 C CNN
@@
 L power:GND #PWR03
 U 1 1 5DD21596
-P 1500 4550
-F 0 "#PWR03" H 1500 4300 50  0001 C CNN
-F 1 "GND" H 1505 4377 50  0000 C CNN
-F 2 "" H 1500 4550 50  0001 C CNN
-F 3 "" H 1500 4550 50  0001 C CNN
-	1    1500 4550
-	1    0    0    -1
-$EndComp
-Wire Wire Line
-	1500 4550 1500 4450
-Wire Wire Line
-	1500 4450 1400 4450
+P 1450 4550
+F 0 "#PWR03" H 1450 4300 50  0001 C CNN
+F 1 "GND" H 1455 4377 50  0000 C CNN
+F 2 "" H 1450 4550 50  0001 C CNN
+F 3 "" H 1450 4550 50  0001 C CNN
+	1    1450 4550
+	1    0    0    -1
+$EndComp
 Wire Wire Line
 	1400 4250 2050 4250
 Connection ~ 2050 4250
-Wire Wire Line
-	1400 4350 1750 4350
 Text Notes 800  1125 0    50   ~ 0
 Battery
@@
 Text Label 3750 2700 0    50   ~ 0
 VREF
-Text Label 1500 4350 0    50   ~ 0
+Text Label 1500 4150 0    50   ~ 0
 RXTX
 $Comp
@@
 RXTX
 Text Label 8850 3550 0    50   ~ 0
+SWDIO
+Text Label 8850 3650 0    50   ~ 0
 SWCLK
-Text Label 8850 3650 0    50   ~ 0
-SWDIO
 Wire Wire Line
 	8800 3650 9350 3650
@@
 	2350 4250 2350 4200
 $Comp
-L Connector_Generic:Conn_01x03 J3
-U 1 1 5E47DF7F
-P 1200 4350
-F 0 "J3" H 1118 4667 50  0000 C CNN
-F 1 "Conn_01x03" H 1118 4576 50  0000 C CNN
-F 2 "Connector_PinHeader_2.54mm:PinHeader_1x03_P2.54mm_Vertical" H 1200 4350 50  0001 C CNN
-F 3 "~" H 1200 4350 50  0001 C CNN
-	1    1200 4350
-	-1   0    0    -1
-$EndComp
-$Comp
 L power:GND #PWR010
 U 1 1 5E4A4D8C
@@
 P 1450 5850
 F 0 "C9" V 1300 5800 50  0000 L CNN
-F 1 "100nF" V 1600 5750 50  0000 L CNN
+F 1 "2.2uF" V 1600 5750 50  0000 L CNN
 F 2 "Capacitor_SMD:C_0402_1005Metric" H 1488 5700 50  0001 C CNN
 F 3 "~" H 1450 5850 50  0001 C CNN
@@
 P 3350 6700
 F 0 "R7" H 3280 6654 50  0000 R CNN
-F 1 "50" H 3280 6745 50  0000 R CNN
+F 1 "1k" H 3280 6745 50  0000 R CNN
 F 2 "Resistor_SMD:R_0402_1005Metric" V 3280 6700 50  0001 C CNN
 F 3 "~" H 3350 6700 50  0001 C CNN
@@
 BLDC motor RPM sensor
 Text Notes 3650 1700 0    55   ~ 11
-Absolute maximum ratings\n———————————————————\nMax. battery input voltage: 50V (12S)\nMax. current: 60A\n\nDC characteristics:\n———————————————————\nInput power supply: 4-10V\nPower consuption: 100mA
+Absolute maximum ratings\n———————————————————\nMax. battery input voltage: 50V (12S)\nMax. current: 60A\n\nDC characteristics:\n———————————————————\nInput power supply: 4-10V\nPower consuption: 20mA
 Wire Notes Line style solid
 	3550 800  5400 800
@@
 Wire Wire Line
 	8200 5150 8200 4950
+$Comp
+L Connector_Generic:Conn_01x03 J3
+U 1 1 5E47DF7F
+P 1200 4250
+F 0 "J3" H 1200 3950 50  0000 C CNN
+F 1 "Conn_01x03" H 1200 4050 50  0000 C CNN
+F 2 "Connector_PinHeader_2.54mm:PinHeader_1x03_P2.54mm_Vertical" H 1200 4250 50  0001 C CNN
+F 3 "~" H 1200 4250 50  0001 C CNN
+	1    1200 4250
+	-1   0    0    1
+$EndComp
+Wire Wire Line
+	1400 4150 1750 4150
+Wire Wire Line
+	1400 4350 1450 4350
+Wire Wire Line
+	1450 4350 1450 4550
 $EndSCHEMATC

Commit message: Replace some components
Parts:
- removed C10, C9: 2.2uF, Capacitor_SMD:C_0402_1005Metric, symbol Device:C
- removed FB1: 120ohm GHz, Resistor_SMD:R_0402_1005Metric, symbol Device:Ferrite_Bead
- removed R7: 1k, Resistor_SMD:R_0402_1005Metric, symbol Device:R
- removed U2: MAX4081S, local:uMAX-8, symbol Amplifier_Current:MAX4081S
- removed U3: STM32G431KBUx, Package_DFN_QFN:QFN-32-1EP_5x5mm_P0.5mm_EP3.45x3.45mm, symbol kapuki:STM32G431KBUx
- removed U4: MCP1501, Package_TO_SOT_SMD:SOT-23-6, symbol kapuki:MCP1501
- added R? (x2): 10k, Resistor_SMD:R_0402_1005Metric, symbol Device:R
- added U3: STM32G431CBTx, Package_QFP:LQFP-48_7x7mm_P0.5mm, symbol kapuki:STM32G431CBTx
- added U?: INA199, Package_SO:SOIC-8_3.9x4.9mm_P1.27mm, symbol kapuki:INA199
Connections:
- wire segments 143 -> 130
- no-connect marks 11 -> 12
Other:
- moved on the sheet: C11, C3, C4, C5, C6, C7, C8, D1, D3, J6, J7, J8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

Commit message: Remove motor RPM measurement capability
Parts:
- removed D1: BZT52H-C3V3, Diode_SMD:D_SOD-123F, symbol Diode:BZT52Bxx
- removed J6: Conn_01x01, Connector_PinSocket_2.54mm:PinSocket_1x01_P2.54mm_Vertical, symbol Connector_Generic:Conn_01x01
- removed R? (x2): 10k, Resistor_SMD:R_0402_1005Metric, symbol Device:R
- added C?: 100nF, Capacitor_SMD:C_0402_1005Metric, symbol Device:C
- added FB?: 100 @ 100MHz, symbol Device:FerriteBead_Small
- R4: value 38k3 0.1% -> 18k 1%
- R5: value 2k4 0.1% -> 2k4 1%
Other:
- note added: "Absolute maximum ratings\n———————————————————\nMax. battery input voltage: 27V (6S)\nMax. current: 60A\n\nDC characteristics:\n———————————————————\nInput power supply: 4-10V\nPower consuption: 20mA"
- note added: "CPU"
- note added: "Power supply & Serial (Jeti EX bus) interface"
- note removed: "Absolute maximum ratings\n———————————————————\nMax. battery input voltage: 50V (12S)\nMax. current: 60A\n\nDC characteristics:\n———————————————————\nInput power supply: 4-10V\nPower consuption: 20mA"
- note removed: "BLDC motor RPM sensor"
- note removed: "Power supply & Jeti EX bus interface"
- note removed: "Voltage reference and power supply for CPU Analog section"
- moved on the sheet: C4, C5, C6, J7, J8
