File: kapuki-cursen-hw.sch (KiCad schematic (older format))
At the start: 27 parts, among them J1 Conn_01x02, J2 Conn_01x02, J3 Conn_01x03, J7 Conn_01x06, J8 Conn_01x05, U1 MIC5235, U3 STM32G431CBTx

Commit message: Add features for the new CPU
Parts:
- U2: renamed from U?; footprint Package_SO:SOIC-8_3.9x4.9mm_P1.27mm -> Package_TO_SOT_SMD:SOT-363_SC-70-6
- gave numbers to parts that had none: 2
Connections:
- net labels added: REF, RX, TX
- net labels removed: MOTORPULSE, VREF
- wire segments 130 -> 128
- no-connect marks 12 -> 30
Other:
- moved on the sheet: D3, R3, R6
Changed lines of the file:
@@
 EESchema Schematic File Version 4
+LIBS:kapuki-cursen-hw-cache
 EELAYER 30 0
 EELAYER END
@@
 	1    0    0    -1
 $EndComp
-Text Label 1500 4150 0    50   ~ 0
+Text Label 1700 4150 2    50   ~ 0
 RXTX
-Text Label 8850 3550 0    50   ~ 0
+Text Label 7250 3550 0    50   ~ 0
 IMEAS
-Text Label 8850 3650 0    50   ~ 0
-MOTORPULSE
-Text Label 9850 4450 0    50   ~ 0
+Text Label 10325 3750 2    50   ~ 0
 RXTX
-Text Label 8850 4850 0    50   ~ 0
+Text Label 9150 4850 2    50   ~ 0
 SWDIO
-Text Label 8850 4950 0    50   ~ 0
+Text Label 9150 4950 2    50   ~ 0
 SWCLK
 Wire Wire Line
-	8800 4950 9350 4950
-Wire Wire Line
-	8800 3650 9350 3650
-Wire Wire Line
-	8800 3550 9350 3550
+	8800 4950 9150 4950
+Wire Wire Line
+	7600 3550 7250 3550
 $Comp
 L Connector_Generic:Conn_01x06 J7
@@
 $EndComp
 Wire Wire Line
-	8800 3950 9350 3950
-Text Label 8850 3950 0    50   ~ 0
-VREF
-Wire Wire Line
-	8800 3850 9350 3850
-Wire Wire Line
-	8800 4050 9350 4050
-Wire Wire Line
-	8800 4150 9350 4150
-Wire Wire Line
-	8800 4250 9350 4250
-Wire Wire Line
-	7600 4050 7250 4050
-Wire Wire Line
-	8800 4350 9350 4350
-Text Label 8850 3850 0    50   ~ 0
+	7600 3750 7250 3750
+Text Label 7250 3750 0    50   ~ 0
 UMEAS
-Text Label 8850 4050 0    50   ~ 0
-EXT1
-Text Label 8850 4150 0    50   ~ 0
-EXT2
-Text Label 8850 4250 0    50   ~ 0
-EXT3
-Text Label 8850 4350 0    50   ~ 0
-EXT5
-Text Label 7500 4050 2    50   ~ 0
-EXT4
 Text Label 4250 5900 0    50   ~ 0
 EXT1
@@
 Wire Wire Line
 	4200 6300 4500 6300
-NoConn ~ 8800 4750
-NoConn ~ 8800 4550
-NoConn ~ 7600 2950
-NoConn ~ 7600 3050
-NoConn ~ 7600 3500
-NoConn ~ 7600 3600
-NoConn ~ 7600 3700
-NoConn ~ 7600 3800
-NoConn ~ 7600 3900
-Wire Wire Line
-	9650 4450 9650 4350
-Text Label 1550 6100 0    50   ~ 0
+Wire Wire Line
+	9950 3750 9950 3650
+Text Label 1850 6100 2    50   ~ 0
 SWCLK
-Text Label 1550 6300 0    50   ~ 0
+Text Label 1850 6300 2    50   ~ 0
 SWDIO
-Text Label 1550 6400 0    50   ~ 0
+Text Label 1850 6400 2    50   ~ 0
 ~RESET~
 Wire Wire Line
@@
 L Device:LED D3
 U 1 1 5DDC9661
-P 10350 3975
-F 0 "D3" V 10389 3858 50  0000 R CNN
-F 1 "LED" V 10298 3858 50  0000 R CNN
-F 2 "LED_SMD:LED_0402_1005Metric" H 10350 3975 50  0001 C CNN
-F 3 "~" H 10350 3975 50  0001 C CNN
-	1    10350 3975
+P 9325 2825
+F 0 "D3" V 9364 2708 50  0000 R CNN
+F 1 "LED" V 9273 2708 50  0000 R CNN
+F 2 "LED_SMD:LED_0402_1005Metric" H 9325 2825 50  0001 C CNN
+F 3 "~" H 9325 2825 50  0001 C CNN
+	1    9325 2825
 	0    -1   -1   0
 $EndComp
@@
 L Device:R R3
 U 1 1 5DDCAC4A
-P 10350 4350
-F 0 "R3" H 10280 4304 50  0000 R CNN
-F 1 "1k" H 10280 4395 50  0000 R CNN
-F 2 "Resistor_SMD:R_0402_1005Metric" V 10280 4350 50  0001 C CNN
-F 3 "~" H 10350 4350 50  0001 C CNN
-	1    10350 4350
+P 9325 3200
+F 0 "R3" H 9255 3154 50  0000 R CNN
+F 1 "1k" H 9255 3245 50  0000 R CNN
+F 2 "Resistor_SMD:R_0402_1005Metric" V 9255 3200 50  0001 C CNN
+F 3 "~" H 9325 3200 50  0001 C CNN
+	1    9325 3200
 	-1   0    0    1
 $EndComp
 Wire Wire Line
-	10350 4200 10350 4125
-Wire Wire Line
-	8800 4850 9350 4850
-NoConn ~ 8800 5050
-Wire Wire Line
-	10350 4500 10350 4650
+	9325 3050 9325 2975
+Wire Wire Line
+	8800 4850 9150 4850
 $Comp
 L power:+3V3 #PWR0101
@@
 Wire Wire Line
 	2250 1550 2250 1450
-Text Label 2600 1550 0    50   ~ 0
+Text Label 2900 1550 2    50   ~ 0
 UMEAS
 $Comp
 L power:+3V3 #PWR0102
 U 1 1 5E3DF860
-P 10350 3750
-F 0 "#PWR0102" H 10350 3600 50  0001 C CNN
-F 1 "+3V3" H 10365 3923 50  0000 C CNN
-F 2 "" H 10350 3750 50  0001 C CNN
-F 3 "" H 10350 3750 50  0001 C CNN
-	1    10350 3750
+P 9325 2600
+F 0 "#PWR0102" H 9325 2450 50  0001 C CNN
+F 1 "+3V3" H 9340 2773 50  0000 C CNN
+F 2 "" H 9325 2600 50  0001 C CNN
+F 3 "" H 9325 2600 50  0001 C CNN
+	1    9325 2600
 	1    0    0    -1
 $EndComp
@@
 $EndComp
 Wire Wire Line
-	10350 3750 10350 3825
-Text Label 6650 2550 2    50   ~ 0
+	9325 2600 9325 2675
+Text Label 6350 2550 0    50   ~ 0
 ~RESET~
 $Comp
@@
 Wire Wire Line
 	2350 4250 2350 4200
-NoConn ~ 8800 3750
 Wire Wire Line
 	1450 6400 1850 6400
@@
 L Device:R R6
 U 1 1 5DD70BDC
-P 9650 4200
-F 0 "R6" H 9580 4154 50  0000 R CNN
-F 1 "4k7" H 9580 4245 50  0000 R CNN
-F 2 "Resistor_SMD:R_0402_1005Metric" V 9580 4200 50  0001 C CNN
-F 3 "~" H 9650 4200 50  0001 C CNN
-	1    9650 4200
+P 9950 3500
+F 0 "R6" H 9880 3454 50  0000 R CNN
+F 1 "4k7" H 9880 3545 50  0000 R CNN
+F 2 "Resistor_SMD:R_0402_1005Metric" V 9880 3500 50  0001 C CNN
+F 3 "~" H 9950 3500 50  0001 C CNN
+	1    9950 3500
 	-1   0    0    1
 $EndComp
@@
 L power:+3V3 #PWR0106
 U 1 1 5E51663B
-P 9650 3900
-F 0 "#PWR0106" H 9650 3750 50  0001 C CNN
-F 1 "+3V3" H 9665 4073 50  0000 C CNN
-F 2 "" H 9650 3900 50  0001 C CNN
-F 3 "" H 9650 3900 50  0001 C CNN
-	1    9650 3900
-	1    0    0    -1
-$EndComp
-Wire Wire Line
-	9650 3900 9650 4050
-Wire Wire Line
-	8800 4650 10350 4650
+P 9950 3200
+F 0 "#PWR0106" H 9950 3050 50  0001 C CNN
+F 1 "+3V3" H 9965 3373 50  0000 C CNN
+F 2 "" H 9950 3200 50  0001 C CNN
+F 3 "" H 9950 3200 50  0001 C CNN
+	1    9950 3200
+	1    0    0    -1
+$EndComp
+Wire Wire Line
+	9950 3200 9950 3350
 Wire Wire Line
 	8400 2350 8400 1750
@@
 $EndComp
 Wire Wire Line
-	8600 1550 8600 1750
+	8600 1550 8600 1625
 Wire Notes Line
 	650  5400 5550 5400
@@
 	1500 6200 1500 6550
 Wire Wire Line
-	8800 4450 9650 4450
-Wire Wire Line
-	9650 4450 10100 4450
-Connection ~ 9650 4450
+	8800 3750 9950 3750
+Wire Wire Line
+	9950 3750 10325 3750
+Connection ~ 9950 3750
 Wire Wire Line
 	4200 5900 4500 5900
@@
 $EndComp
 Wire Wire Line
-	1400 4150 1750 4150
+	1400 4150 1700 4150
 Wire Wire Line
 	1400 4350 1450 4350
@@
 	1450 4350 1450 4550
 $Comp
-L kapuki:INA199 U?
+L kapuki:INA199 U2
 U 1 1 601AB1BB
 P 3250 2600
-F 0 "U?" H 3400 2700 50  0000 L CNN
+F 0 "U2" H 3400 2700 50  0000 L CNN
 F 1 "INA199" H 3400 2500 50  0000 L CNN
-F 2 "Package_SO:SOIC-8_3.9x4.9mm_P1.27mm" H 3250 1950 50  0001 C CNN
+F 2 "Package_TO_SOT_SMD:SOT-363_SC-70-6" H 3250 1950 50  0001 C CNN
 F 3 "https://www.ti.com/lit/ds/symlink/ina199.pdf" H 3400 2750 50  0001 C CNN
 	1    3250 2600
@@
 $EndComp
 $Comp
-L power:VCC #PWR?
+L power:VCC #PWR0105
 U 1 1 601D6C1D
 P 3200 2100
-F 0 "#PWR?" H 3200 1950 50  0001 C CNN
+F 0 "#PWR0105" H 3200 1950 50  0001 C CNN
 F 1 "VCC" H 3215 2273 50  0000 C CNN
 F 2 "" H 3200 2100 50  0001 C CNN
@@
 	3200 2100 3200 2300
 $Comp
-L power:GND #PWR?
+L power:GND #PWR0107
 U 1 1 601DC898
 P 3200 3100
-F 0 "#PWR?" H 3200 2850 50  0001 C CNN
+F 0 "#PWR0107" H 3200 2850 50  0001 C CNN
 F 1 "GND" H 3205 2927 50  0000 C CNN
 F 2 "" H 3200 3100 50  0001 C CNN
@@
 IMEAS
 Text Label 3800 2950 2    50   ~ 0
-VREF
+REF
 $Comp
 L kapuki:STM32G431CBTx U3
@@
 	8000 5300 8100 5300
 Connection ~ 8100 5300
-NoConn ~ 8000 2350
-$Comp
-L power:GND #PWR?
+$Comp
+L power:GND #PWR0111
 U 1 1 602C6333
 P 7150 4400
-F 0 "#PWR?" H 7150 4150 50  0001 C CNN
+F 0 "#PWR0111" H 7150 4150 50  0001 C CNN
 F 1 "GND" H 7155 4227 50  0000 C CNN
 F 2 "" H 7150 4400 50  0001 C CNN
@@
 	2150 2700 3000 2700
 $Comp
-L Device:C C?
+L Device:C C9
 U 1 1 60325E74
 P 7650 1950
-F 0 "C?" H 7765 1996 50  0000 L CNN
+F 0 "C9" H 7765 1996 50  0000 L CNN
 F 1 "100nF" H 7765 1905 50  0000 L CNN
 F 2 "Capacitor_SMD:C_0402_1005Metric" H 7688 1800 50  0001 C CNN
@@
 	8200 2300 8100 2300
 $Comp
-L Device:FerriteBead_Small FB?
+L Device:FerriteBead_Small FB1
 U 1 1 6036CA8B
 P 8250 1750
-F 0 "FB?" V 8013 1750 50  0000 C CNN
+F 0 "FB1" V 8013 1750 50  0000 C CNN
 F 1 "100 @ 100MHz" V 8104 1750 50  0000 C CNN
 F 2 "" V 8180 1750 50  0001 C CNN
@@
 Text Notes 8150 6000 0    79   ~ 16
 CPU
+NoConn ~ 8000 2350
+Wire Wire Line
+	8800 4450 9150 4450
+Text Label 9150 4450 2    50   ~ 0
+TX
+Wire Wire Line
+	8800 4550 9150 4550
+Text Label 9150 4550 2    50   ~ 0
+RX
+Wire Wire Line
+	8800 4050 9150 4050
+Text Label 9150 4050 2    50   ~ 0
+REF
+Wire Wire Line
+	8800 3550 9325 3550
+Wire Wire Line
+	9325 3350 9325 3550
+NoConn ~ 8800 5050
+NoConn ~ 8800 4750
+NoConn ~ 8800 4350
+NoConn ~ 8800 4250
+NoConn ~ 8800 4150
+NoConn ~ 8800 3950
+NoConn ~ 8800 3850
+NoConn ~ 8800 3650
+NoConn ~ 8800 2950
+NoConn ~ 7600 2750
+NoConn ~ 7600 2850
+NoConn ~ 7600 2950
+NoConn ~ 7600 3150
+NoConn ~ 7600 3250
+NoConn ~ 7600 3350
+NoConn ~ 7600 3650
+NoConn ~ 7600 3850
+NoConn ~ 7600 3950
+NoConn ~ 7600 4050
+NoConn ~ 7600 4150
+NoConn ~ 7600 4250
+NoConn ~ 7600 4450
+NoConn ~ 7600 4550
+NoConn ~ 7600 4650
+NoConn ~ 7600 4750
+NoConn ~ 7600 4850
+NoConn ~ 7600 4950
+NoConn ~ 7600 5050
+$Comp
+L power:PWR_FLAG #FLG0102
+U 1 1 61547996
+P 8775 1625
+F 0 "#FLG0102" H 8775 1700 50  0001 C CNN
+F 1 "PWR_FLAG" V 8775 1925 50  0000 C CNN
+F 2 "" H 8775 1625 50  0001 C CNN
+F 3 "~" H 8775 1625 50  0001 C CNN
+	1    8775 1625
+	0    1    1    0
+$EndComp
+Wire Wire Line
+	8775 1625 8600 1625
+Connection ~ 8600 1625
+Wire Wire Line
+	8600 1625 8600 1750
+NoConn ~ 8800 4650
 $EndSCHEMATC

Commit message: Start the rev. 4 PCb design
Parts:
- added C10: 100n, Capacitor_SMD:C_0603_1608Metric_Pad1.08x0.95mm_HandSolder, symbol Device:C
- C1, C11, C2, C3, C4, C5, C6, C7, C8, C9: footprint Capacitor_SMD:C_0402_1005Metric -> Capacitor_SMD:C_0603_1608Metric_Pad1.08x0.95mm_HandSolder
- D3: footprint LED_SMD:LED_0402_1005Metric -> LED_SMD:LED_0603_1608Metric_Pad1.05x0.95mm_HandSolder
- FB1: footprint (none) -> Inductor_SMD:L_0603_1608Metric_Pad1.05x0.95mm_HandSolder
- J7: footprint Connector_PinSocket_2.54mm:PinSocket_1x06_P2.54mm_Vertical -> Connector_PinSocket_1.27mm:PinSocket_1x06_P1.27mm_Vertical
- J8: footprint Connector_JST:JST_SH_BM05B-SRSS-TB_1x05-1MP_P1.00mm_Vertical -> local:TestPoint_5Pad_D0.8mm
- R2, R3, R4, R5, R6, R8: footprint Resistor_SMD:R_0402_1005Metric -> Resistor_SMD:R_0603_1608Metric_Pad0.98x0.95mm_HandSolder
Connections:
- wire segments 128 -> 132
Changed lines of the file:
@@
 EESchema Schematic File Version 4
-LIBS:kapuki-cursen-hw-cache
 EELAYER 30 0
 EELAYER END
@@
 F 0 "R2" V 3950 2600 50  0000 C CNN
 F 1 "1k" V 4050 2600 50  0000 C CNN
-F 2 "Resistor_SMD:R_0402_1005Metric" V 3980 2600 50  0001 C CNN
+F 2 "Resistor_SMD:R_0603_1608Metric_Pad0.98x0.95mm_HandSolder" V 3980 2600 50  0001 C CNN
 F 3 "~" H 4050 2600 50  0001 C CNN
 	1    4050 2600
@@
 F 0 "C3" H 4515 2846 50  0000 L CNN
 F 1 "100pF" H 4515 2755 50  0000 L CNN
-F 2 "Capacitor_SMD:C_0402_1005Metric" H 4438 2650 50  0001 C CNN
+F 2 "Capacitor_SMD:C_0603_1608Metric_Pad1.08x0.95mm_HandSolder" H 4438 2650 50  0001 C CNN
 F 3 "~" H 4400 2800 50  0001 C CNN
 	1    4400 2800
@@
 F 0 "C2" H 3515 4496 50  0000 L CNN
 F 1 "2.2uF" H 3515 4405 50  0000 L CNN
-F 2 "Capacitor_SMD:C_0402_1005Metric" H 3438 4300 50  0001 C CNN
+F 2 "Capacitor_SMD:C_0603_1608Metric_Pad1.08x0.95mm_HandSolder" H 3438 4300 50  0001 C CNN
 F 3 "~" H 3400 4450 50  0001 C CNN
 	1    3400 4450
@@
 F 0 "C1" H 2165 4496 50  0000 L CNN
 F 1 "1.0uF" H 2165 4405 50  0000 L CNN
-F 2 "Capacitor_SMD:C_0402_1005Metric" H 2088 4300 50  0001 C CNN
+F 2 "Capacitor_SMD:C_0603_1608Metric_Pad1.08x0.95mm_HandSolder" H 2088 4300 50  0001 C CNN
 F 3 "~" H 2050 4450 50  0001 C CNN
 	1    2050 4450
@@
 F 0 "J7" H 4000 5800 50  0000 C CNN
 F 1 "Conn_01x06" H 3918 5766 50  0001 C CNN
-F 2 "Connector_PinSocket_2.54mm:PinSocket_1x06_P2.54mm_Vertical" H 4000 6200 50  0001 C CNN
+F 2 "Connector_PinSocket_1.27mm:PinSocket_1x06_P1.27mm_Vertical" H 4000 6200 50  0001 C CNN
 F 3 "~" H 4000 6200 50  0001 C CNN
 	1    4000 6200
@@
 F 0 "R4" H 2180 1254 50  0000 R CNN
 F 1 "18k 1%" H 2180 1345 50  0000 R CNN
-F 2 "Resistor_SMD:R_0402_1005Metric" V 2180 1300 50  0001 C CNN
+F 2 "Resistor_SMD:R_0603_1608Metric_Pad0.98x0.95mm_HandSolder" V 2180 1300 50  0001 C CNN
 F 3 "~" H 2250 1300 50  0001 C CNN
 	1    2250 1300
@@
 F 0 "R5" H 2180 1704 50  0000 R CNN
 F 1 "2k4 1%" H 2180 1795 50  0000 R CNN
-F 2 "Resistor_SMD:R_0402_1005Metric" V 2180 1750 50  0001 C CNN
+F 2 "Resistor_SMD:R_0603_1608Metric_Pad0.98x0.95mm_HandSolder" V 2180 1750 50  0001 C CNN
 F 3 "~" H 2250 1750 50  0001 C CNN
 	1    2250 1750
@@
 F 0 "D3" V 9364 2708 50  0000 R CNN
 F 1 "LED" V 9273 2708 50  0000 R CNN
-F 2 "LED_SMD:LED_0402_1005Metric" H 9325 2825 50  0001 C CNN
+F 2 "LED_SMD:LED_0603_1608Metric_Pad1.05x0.95mm_HandSolder" H 9325 2825 50  0001 C CNN
 F 3 "~" H 9325 2825 50  0001 C CNN
 	1    9325 2825
@@
 F 0 "R3" H 9255 3154 50  0000 R CNN
 F 1 "1k" H 9255 3245 50  0000 R CNN
-F 2 "Resistor_SMD:R_0402_1005Metric" V 9255 3200 50  0001 C CNN
+F 2 "Resistor_SMD:R_0603_1608Metric_Pad0.98x0.95mm_HandSolder" V 9255 3200 50  0001 C CNN
 F 3 "~" H 9325 3200 50  0001 C CNN
 	1    9325 3200
@@
 F 0 "J8" H 1250 6500 50  0000 C CNN
 F 1 "Conn_01x05" H 1168 5866 50  0001 C CNN
-F 2 "Connector_JST:JST_SH_BM05B-SRSS-TB_1x05-1MP_P1.00mm_Vertical" H 1250 6200 50  0001 C CNN
+F 2 "local:TestPoint_5Pad_D0.8mm" H 1250 6200 50  0001 C CNN
 F 3 "~" H 1250 6200 50  0001 C CNN
 	1    1250 6200
@@
 F 0 "C6" H 7315 1996 50  0000 L CNN
 F 1 "100nF" H 7315 1905 50  0000 L CNN
-F 2 "Capacitor_SMD:C_0402_1005Metric" H 7238 1800 50  0001 C CNN
+F 2 "Capacitor_SMD:C_0603_1608Metric_Pad1.08x0.95mm_HandSolder" H 7238 1800 50  0001 C CNN
 F 3 "~" H 7200 1950 50  0001 C CNN
 	1    7200 1950
@@
 F 0 "C5" H 6865 1996 50  0000 L CNN
 F 1 "100nF" H 6865 1905 50  0000 L CNN
-F 2 "Capacitor_SMD:C_0402_1005Metric" H 6788 1800 50  0001 C CNN
+F 2 "Capacitor_SMD:C_0603_1608Metric_Pad1.08x0.95mm_HandSolder" H 6788 1800 50  0001 C CNN
 F 3 "~" H 6750 1950 50  0001 C CNN
 	1    6750 1950
@@
 F 0 "C4" H 6415 1996 50  0000 L CNN
 F 1 "4.7uF" H 6415 1905 50  0000 L CNN
-F 2 "Capacitor_SMD:C_0402_1005Metric" H 6338 1800 50  0001 C CNN
+F 2 "Capacitor_SMD:C_0603_1608Metric_Pad1.08x0.95mm_HandSolder" H 6338 1800 50  0001 C CNN
 F 3 "~" H 6300 1950 50  0001 C CNN
 	1    6300 1950
@@
 F 0 "R6" H 9880 3454 50  0000 R CNN
 F 1 "4k7" H 9880 3545 50  0000 R CNN
-F 2 "Resistor_SMD:R_0402_1005Metric" V 9880 3500 50  0001 C CNN
+F 2 "Resistor_SMD:R_0603_1608Metric_Pad0.98x0.95mm_HandSolder" V 9880 3500 50  0001 C CNN
 F 3 "~" H 9950 3500 50  0001 C CNN
 	1    9950 3500
@@
 F 0 "C8" H 9115 1996 50  0000 L CNN
 F 1 "10nF" H 9115 1905 50  0000 L CNN
-F 2 "Capacitor_SMD:C_0402_1005Metric" H 9038 1800 50  0001 C CNN
+F 2 "Capacitor_SMD:C_0603_1608Metric_Pad1.08x0.95mm_HandSolder" H 9038 1800 50  0001 C CNN
 F 3 "~" H 9000 1950 50  0001 C CNN
 	1    9000 1950
@@
 F 0 "C7" H 8715 1996 50  0000 L CNN
 F 1 "1uF" H 8715 1905 50  0000 L CNN
-F 2 "Capacitor_SMD:C_0402_1005Metric" H 8638 1800 50  0001 C CNN
+F 2 "Capacitor_SMD:C_0603_1608Metric_Pad1.08x0.95mm_HandSolder" H 8638 1800 50  0001 C CNN
 F 3 "~" H 8600 1950 50  0001 C CNN
 	1    8600 1950
@@
 F 0 "C11" H 6875 2800 50  0000 L CNN
 F 1 "100nF" H 6875 2700 50  0000 L CNN
-F 2 "Capacitor_SMD:C_0402_1005Metric" H 6788 2600 50  0001 C CNN
+F 2 "Capacitor_SMD:C_0603_1608Metric_Pad1.08x0.95mm_HandSolder" H 6788 2600 50  0001 C CNN
 F 3 "~" H 6750 2750 50  0001 C CNN
 	1    6750 2750
@@
 $EndComp
 Wire Wire Line
-	3200 2100 3200 2300
+	3200 2100 3200 2200
 $Comp
 L power:GND #PWR0107
@@
 F 0 "C9" H 7765 1996 50  0000 L CNN
 F 1 "100nF" H 7765 1905 50  0000 L CNN
-F 2 "Capacitor_SMD:C_0402_1005Metric" H 7688 1800 50  0001 C CNN
+F 2 "Capacitor_SMD:C_0603_1608Metric_Pad1.08x0.95mm_HandSolder" H 7688 1800 50  0001 C CNN
 F 3 "~" H 7650 1950 50  0001 C CNN
 	1    7650 1950
@@
 F 0 "FB1" V 8013 1750 50  0000 C CNN
 F 1 "100 @ 100MHz" V 8104 1750 50  0000 C CNN
-F 2 "" V 8180 1750 50  0001 C CNN
+F 2 "Inductor_SMD:L_0603_1608Metric_Pad1.05x0.95mm_HandSolder" V 8180 1750 50  0001 C CNN
 F 3 "~" H 8250 1750 50  0001 C CNN
 	1    8250 1750
@@
 F 0 "R8" V 7425 4400 50  0000 R CNN
 F 1 "10k" V 7346 4421 50  0000 R CNN
-F 2 "Resistor_SMD:R_0402_1005Metric" V 7280 4350 50  0001 C CNN
+F 2 "Resistor_SMD:R_0603_1608Metric_Pad0.98x0.95mm_HandSolder" V 7280 4350 50  0001 C CNN
 F 3 "~" H 7350 4350 50  0001 C CNN
 	1    7350 4350
@@
 	8600 1625 8600 1750
 NoConn ~ 8800 4650
+$Comp
+L Device:C C10
+U 1 1 6040DBB1
+P 3450 2200
+F 0 "C10" V 3198 2200 50  0000 C CNN
+F 1 "100n" V 3289 2200 50  0000 C CNN
+F 2 "Capacitor_SMD:C_0603_1608Metric_Pad1.08x0.95mm_HandSolder" H 3488 2050 50  0001 C CNN
+F 3 "~" H 3450 2200 50  0001 C CNN
+	1    3450 2200
+	0    1    1    0
+$EndComp
+Wire Wire Line
+	3200 2200 3300 2200
+Connection ~ 3200 2200
+Wire Wire Line
+	3200 2200 3200 2300
+$Comp
+L power:GND #PWR04
+U 1 1 604129DA
+P 3700 2300
+F 0 "#PWR04" H 3700 2050 50  0001 C CNN
+F 1 "GND" H 3705 2127 50  0000 C CNN
+F 2 "" H 3700 2300 50  0001 C CNN
+F 3 "" H 3700 2300 50  0001 C CNN
+	1    3700 2300
+	1    0    0    -1
+$EndComp
+Wire Wire Line
+	3600 2200 3700 2200
+Wire Wire Line
+	3700 2200 3700 2300
 $EndSCHEMATC
