File: kapuki-cursen-hw.kicad_pcb (KiCad board)
At the start: 4 copper layers, 27.9 x 19 mm, 28 parts, among them J1 Conn_01x02, J2 Conn_01x02, J3 Conn_01x03, J7 Conn_01x06, J8 Conn_01x05, U1 MIC5235, U2 INA199, U3 STM32G431CBTx

Commit message: rev. 4 routing is almost finished
Parts:
- added REF**: OSHW-Logo2_7.3x6mm_SilkScreen, Symbol:OSHW-Logo2_7.3x6mm_SilkScreen, F.Cu at (137.5, 78.4)
- added SW1: BOOT, Button_Switch_SMD:Panasonic_EVQPUJ_EVQPUA, F.Cu at (109.2, 83.6)
- J7: value Conn_01x06 -> Conn_01x03; footprint Connector_PinSocket_1.27mm:PinSocket_1x06_P1.27mm_Vertical -> Connector_PinHeader_2.54mm:PinHeader_1x03_P2.54mm_Vertical
- moved J7 56.7 mm to (122.7, 91.4), turned to 90 degrees
- moved D3 9.38 mm to (138.9, 82.8), turned to 270 degrees
- moved R3 8.21 mm to (136.9, 82.8), turned to 90 degrees
- moved U2 7.59 mm to (142.3, 77.4), turned to 90 degrees
- moved C10 6.88 mm to (142.6, 79.9), turned to 0 degrees
- moved FB1 6.25 mm to (125.6, 77.4), turned to 270 degrees
- moved R2 6.00 mm to (140.7, 74.8), turned to 0 degrees
- moved C3 5.40 mm to (137.2, 74.8), turned to 180 degrees
- moved J8 4.33 mm to (132.3, 91.2)
- moved C2 4.13 mm to (141.5, 84.1)
- moved U1 4.06 mm to (144.5, 84.1)
- moved C1 3.82 mm to (144.8, 86.9)
- moved C5 2.92 mm to (124.2, 85.6), turned to 90 degrees
- moved R5 1.27 mm to (130.3, 74.7)
- moved C4 1.08 mm to (122.4, 85.6), turned to 90 degrees
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Connections:
- J7 pad 2: /EXT5 -> /TX
- J7 pad 3: /EXT4 -> /RX
Routing:
- net GND: track 0.00 -> 31.4 mm, vias 0 -> 35
- net +3V3: track 0.00 -> 22.7 mm, vias 0 -> 10
- net /TX: track 0.00 -> 17.6 mm, vias 0 -> 1
- net /RXTX: track 0.00 -> 14.7 mm, vias 0 -> 1
- net /IMEAS: track 0.00 -> 12.3 mm
- net /~RESET~: track 0.00 -> 12.2 mm, vias 0 -> 1
- net /SWDIO: track 0.00 -> 11.1 mm
- net Net-(R1-Pad2): track 0.00 -> 10.4 mm, vias 0 -> 1
- net VCC: track 0.00 -> 10.3 mm
- net /UMEAS: track 0.00 -> 9.77 mm
- net /REF: track 0.00 -> 9.43 mm
- net /RX: track 0.00 -> 8.74 mm, vias 0 -> 1
- net VDDA: track 0.00 -> 8.52 mm
- net Net-(R1-Pad3): track 0.00 -> 7.57 mm, vias 0 -> 1
- net /SWCLK: track 0.00 -> 7.41 mm
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- added copper zone on In2.Cu, net +3V3
- added copper zone on B.Cu, net GND
- added copper zone on F.Cu, net GND
- added copper zone on In1.Cu, net GND
- added copper zone on B.Cu, net Net-(J1-Pad2)
- added copper zone on B.Cu, net Net-(J2-Pad2)
Other:
- board size 27.9 x 19 mm -> 27.9 x 19.8 mm
- board text added: "G"
- board text added: "R"
- board text added: "T"
- board text added: "UART"
- board text added: "rev. 4, 2105"
- board text removed: "SWD"
- board text removed: "rev. 4 2106"

Commit message: Finished rev. 4
Parts:
- SW1: footprint Button_Switch_SMD:Panasonic_EVQPUJ_EVQPUA -> Button_Switch_SMD:SW_SPST_PTS810; moved to B.Cu
- moved SW1 26.3 mm to (134.4, 91.2)
- moved C1 0.38 mm to (144.4, 87.0), turned to 0 degrees
Connections:
- C10 pad 2: VCC -> +3V3
- U2 pad 3: VCC -> +3V3
Routing:
- net +3V3: track 22.7 -> 35.5 mm, vias 10 -> 12
- net Net-(R8-Pad2): track 2.45 -> 11.6 mm
- net GND: track 31.4 -> 40.1 mm, vias 35 -> 36
Other:
- net class VCC removed
- rule via_min_drill: 0.3302 -> 0.254
- rule via_min_size: 0.6858 -> 0.508
- board text added: "2105"
- board text added: "3"
- board text added: "BOOT"
- board text added: "C"
- board text added: "D"
- board text added: "RX"
- board text added: "TX"
- board text added: "rev. 4"
- board text removed: "R"
- board text removed: "T"
- board text removed: "rev. 4, 2105"
